Commit message: update mesh

File: urdf/bck_agv.xacro (robot description, xacro)
@@ -90,5 +90,5 @@
   </collision>
 </link>
-<link name="lidar_1">
+<!-- <link name="lidar_1">
   <inertial>
     <origin xyz="-0.0016067454834169381 -2.980464184150879e-05 0.010665743146427403" rpy="0 0 0"/>
@@ -109,5 +109,5 @@
     </geometry>
   </collision>
-</link>
+</link> -->
 <joint name="base_link_arti_dis" type="fixed">
   <origin xyz="-0.24 0.0 0.385" rpy="0 0 0"/>
@@ -119,5 +119,5 @@
   <parent link="base_link"/>
   <child link="TekerSag_1"/>
-  <axis xyz="0.0 1.0 -0.0"/>
+  <axis xyz="0.0 -1.0 0.0"/>
 </joint>
 <joint name="sol_teker_vel_motor" type="continuous">
@@ -127,8 +127,8 @@
   <axis xyz="0.0 1.0 0.0"/>
 </joint>
-<joint name="lidar" type="fixed">
+<!-- <joint name="lidar" type="fixed">
   <origin xyz="0.343626 0.000924 0.1976" rpy="0 0 0"/>
   <parent link="base_link"/>
   <child link="lidar_1"/>
-</joint>
+</joint> -->
 </robot>

Commit message: diff drive fix

File: urdf/bck_agv.xacro (robot description, xacro)
@@ -119,5 +119,5 @@
   <parent link="base_link"/>
   <child link="TekerSag_1"/>
-  <axis xyz="0.0 -1.0 0.0"/>
+  <axis xyz="0.0 1.0 0.0"/>
 </joint>
 <joint name="sol_teker_vel_motor" type="continuous">
